File: PCB/PCB-Sprint.kicad_pcb (KiCad board)
At the start: 2 copper layers, 384 x 64 mm, 22 parts

Commit message: commit
Parts:
- added G***: LOGO, 1_PCB-Sprint:8_Fsilk, F.Cu at (240.0, 107.0)
- added G***: LOGO, 1_PCB-Sprint:6_Fsilk, F.Cu at (176.0, 108.0)
- added G***: LOGO, 1_PCB-Sprint:5_Fsilk, F.Cu at (112.0, 107.0)
- added Prakshab: LOGO, 1_PCB-Sprint:14_Fsilk, F.Cu at (304.0, 107.0)
- Hello :): renamed from REF**
- moved REF** 17.0 mm to (159.0, 106.0)
- moved REF** 15.3 mm to (253.1, 99.0)
- moved REF** 8.94 mm to (56.0, 103.0)
- moved REF** 7.07 mm to (305.0, 114.0)
Routing:
- net (no net): track 0.50 -> 223.9 mm, vias 0 -> 2
- removed copper zone on F.Cu, net (none)
Other:
- outline, holes or cut-outs redrawn
- board text added: "Adhikari"
- board text added: "https://github.com/coolerzanu"

Commit message: commit
Routing:
- added copper zone on B.Cu, net (none)
- added copper zone on F.Cu, net (none)
Changed lines of the file:
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@@
 			(drillshape 0)
 			(scaleselection 1)
-			(outputdirectory "../../../../Downloads/FINAL FINAL FINAL/")
+			(outputdirectory "../../../../Downloads/FINAL FINAL FINAL FINAL/")
 		)
 	)
@@
 		(net "")
 	)
+	(zone
+		(layer "F.Cu")
+		(hatch edge 0.5)
+		(priority 1)
+		(connect_pads
+			(clearance 0.5)
+		)
+		(min_thickness 0.25)
+		(fill yes
+			(thermal_gap 0.5)
+			(thermal_bridge_width 0.5)
+			(island_removal_mode 1)
+		)
+		(polygon
+			(pts
+				(xy 16 71) (xy 351 71) (xy 347 157) (xy 16 151)
+			)
+		)
+	)
+	(zone
+		(layers "F.Cu" "B.Cu")
+		(hatch edge 0.5)
+		(connect_pads
+			(clearance 0.5)
+		)
+		(min_thickness 0.25)
+		(fill yes
+			(thermal_gap 0.5)
+			(thermal_bridge_width 0.5)
+			(island_removal_mode 1)
+		)
+		(polygon
+			(pts
+				(xy -53 72) (xy 15 71) (xy 16 71) (xy 16 145) (xy -53 144)
+			)
+		)
+	)
 	(group ""
